File: ui_daughterboard/ui_daughterboard.kicad_sch (KiCad schematic)
At the start: 13 parts, among them J101 Conn_01x06_Male, J102 Conn_01x10_Male, J103 Conn_01x04_Female, SW101 SW_MEC_5E, SW102 SW_MEC_5E

Commit message: final pcb? about to copy layout for daughterboard
Connections:
- net TEST_BLIPPER_P3: now reaches J102.9 (Pin_9)
- no-connect marks 1 -> 0
Other:
- note added: "Connector receives the 8 microdrive LED signals from the Pico's GPIOs. The common return goes back to its current limiting resistor via the same connector. This connector is part of the physical structure of the 2 boards, and matches up with J301 on the main PCB."
- note added: "OLED signals come in from main board. Switch signals go back. Common ground and VCC connect here too. This connector is part of the physical structure of the 2 boards, and matches up with J302 on the main PCB."
- note added: "There's no OLED footprint as such, so using a 4 hole connector matching OLED input pins. Make sure it's the right way round on the PCB!"
- note removed: "Connector receives the 8 microdrive LED signals from the Pico's GPIOs. The common return goes back to its current limiting resistor via the same connector."
- note removed: "OLED signals come in from main board. Switch signals go back."
- note removed: "There's no OLED footprint as such, so using a 4 hole connector matching OLED input pins"
- moved on the sheet: J101, J102

Commit message: lots more work to finalise the board pre-fab
Parts:
- removed SW101, SW102: SW_MEC_5E, Button_Switch_THT:SW_PUSH_6mm_H4.3mm, symbol Switch:SW_MEC_5E
- added SW101, SW102: SW_SPST, Button_Switch_THT:SW_PUSH_6mm_H4.3mm, symbol Switch:SW_SPST
- added TP101: TestPoint, TestPoint:TestPoint_THTPad_D2.0mm_Drill1.0mm, symbol Connector:TestPoint
- J101: footprint (none) -> Connector_PinHeader_2.54mm:PinHeader_1x06_P2.54mm_Vertical
- J102: footprint (none) -> Connector_PinHeader_2.54mm:PinHeader_1x10_P2.54mm_Vertical
- J103: footprint (none) -> Connector_PinHeader_2.54mm:PinHeader_1x04_P2.54mm_Vertical
Connections:
- net ACTION_SW: now also SW101.1 (A)
- net CANCEL_SW: now also SW102.1 (A)
- net GND: now also SW101.2 (B), SW102.2 (B)
- net TEST_BLIPPER_P3: now also TP101.1
Changed lines of the file:
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@@
   (title_block
     (title "User Interface Daughterboard")
-    (date "2023-06-19")
+    (date "2023-06-23")
     (rev "v1.0WIP")
   )
-  (junction (at 150.368 37.846) (diameter 0) (color 0 0 0 0)
-  )
   (junction (at 57.912 53.34) (diameter 0) (color 0 0 0 0)
   )
-  (junction (at 140.208 37.846) (diameter 0) (color 0 0 0 0)
-  )
   (junction (at 57.912 27.94) (diameter 0) (color 0 0 0 0)
   )
   (junction (at 57.912 40.132) (diameter 0) (color 0 0 0 0)
   )
-  (junction (at 182.88 37.592) (diameter 0) (color 0 0 0 0)
-  )
-  (junction (at 172.72 37.592) (diameter 0) (color 0 0 0 0)
-  )
   (junction (at 57.912 66.802) (diameter 0) (color 0 0 0 0)
   )
@@
     (stroke (width 0) (type default) (color 0 0 0 0))
   )
-  (wire (pts (xy 182.88 35.052) (xy 182.88 37.592))
+  (wire (pts (xy 182.88 35.052) (xy 182.88 43.18))
     (stroke (width 0) (type default) (color 0 0 0 0))
   )
@@
     (stroke (width 0) (type default) (color 0 0 0 0))
   )
+  (wire (pts (xy 209.804 69.342) (xy 209.804 71.628))
+    (stroke (width 0) (type default) (color 0 0 0 0))
+  )
   (wire (pts (xy 140.208 37.846) (xy 137.16 37.846))
     (stroke (width 0) (type default) (color 0 0 0 0))
@@
     (stroke (width 0) (type default) (color 0 0 0 0))
   )
-  (wire (pts (xy 150.368 37.846) (xy 150.368 43.18))
-    (stroke (width 0) (type default) (color 0 0 0 0))
-  )
   (wire (pts (xy 110.49 156.718) (xy 144.78 156.718))
     (stroke (width 0) (type default) (color 0 0 0 0))
@@
     (stroke (width 0) (type default) (color 0 0 0 0))
   )
-  (wire (pts (xy 182.88 37.592) (xy 182.88 43.18))
-    (stroke (width 0) (type default) (color 0 0 0 0))
-  )
   (wire (pts (xy 137.922 68.834) (xy 130.302 68.834))
     (stroke (width 0) (type default) (color 0 0 0 0))
@@
     (stroke (width 0) (type default) (color 0 0 0 0))
   )
-  (wire (pts (xy 150.368 35.306) (xy 150.368 37.846))
+  (wire (pts (xy 150.368 35.306) (xy 150.368 43.18))
     (stroke (width 0) (type default) (color 0 0 0 0))
   )
@@
     )
   )
+  (global_label "TEST_BLIPPER_P3" (shape input) (at 209.804 71.628 0) (fields_autoplaced)
+    (effects (font (size 1.27 1.27)) (justify left))
+    (property "Intersheet References" "${INTERSHEET_REFS}" (id 0) (at 228.7876 71.5486 0)
+      (effects (font (size 1.27 1.27)) (justify left) hide)
+    )
+  )
   (global_label "OLED_SDA" (shape input) (at 155.702 71.374 180) (fields_autoplaced)
     (effects (font (size 1.27 1.27)) (justify right))
@@
     (property "Reference" "J102" (id 0) (at 52.959 139.446 0))
     (property "Value" "Conn_01x10_Male" (id 1) (at 52.959 141.986 0))
-    (property "Footprint" "" (id 2) (at 52.324 154.94 0)
+    (property "Footprint" "Connector_PinHeader_2.54mm:PinHeader_1x10_P2.54mm_Vertical" (id 2) (at 52.324 154.94 0)
       (effects (font (size 1.27 1.27)) hide)
     )
@@
       (effects (font (size 1.27 1.27)) (justify left))
     )
-    (property "Footprint" "" (id 2) (at 160.782 66.294 0)
+    (property "Footprint" "Connector_PinHeader_2.54mm:PinHeader_1x04_P2.54mm_Vertical" (id 2) (at 160.782 66.294 0)
       (effects (font (size 1.27 1.27)) hide)
     )
@@
     (pin "3")
     (pin "4")
+  )
+  (symbol (lib_id "Switch:SW_SPST") (at 145.288 35.306 0) (unit 1)
+    (in_bom yes) (on_board yes) (fields_autoplaced)
+    (property "Reference" "SW101" (id 0) (at 145.288 28.956 0))
+    (property "Value" "SW_SPST" (id 1) (at 145.288 31.496 0))
+    (property "Footprint" "Button_Switch_THT:SW_PUSH_6mm_H4.3mm" (id 2) (at 145.288 35.306 0)
+      (effects (font (size 1.27 1.27)) hide)
+    )
+    (property "Datasheet" "~" (id 3) (at 145.288 35.306 0)
+      (effects (font (size 1.27 1.27)) hide)
+    )
+    (pin "1")
+    (pin "2")
   )
   (symbol (lib_id "Device:LED_Small") (at 48.006 40.132 180) (unit 1)
@@
     (pin "2")
   )
+  (symbol (lib_id "Switch:SW_SPST") (at 177.8 35.052 0) (unit 1)
+    (in_bom yes) (on_board yes) (fields_autoplaced)
+    (property "Reference" "SW102" (id 0) (at 177.8 28.702 0))
+    (property "Value" "SW_SPST" (id 1) (at 177.8 31.242 0))
+    (property "Footprint" "Button_Switch_THT:SW_PUSH_6mm_H4.3mm" (id 2) (at 177.8 35.052 0)
+      (effects (font (size 1.27 1.27)) hide)
+    )
+    (property "Datasheet" "~" (id 3) (at 177.8 35.052 0)
+      (effects (font (size 1.27 1.27)) hide)
+    )
+    (pin "1")
+    (pin "2")
+  )
   (symbol (lib_id "Device:LED_Small") (at 48.514 66.802 180) (unit 1)
     (in_bom yes) (on_board yes) (fields_autoplaced)
@@
     (pin "2")
   )
-  (symbol (lib_id "Switch:SW_MEC_5E") (at 145.288 37.846 0) (unit 1)
-    (in_bom yes) (on_board yes) (fields_autoplaced)
-    (property "Reference" "SW101" (id 0) (at 145.288 27.432 0))
-    (property "Value" "SW_MEC_5E" (id 1) (at 145.288 29.972 0))
-    (property "Footprint" "Button_Switch_THT:SW_PUSH_6mm_H4.3mm" (id 2) (at 145.288 30.226 0)
-      (effects (font (size 1.27 1.27)) hide)
-    )
-    (property "Datasheet" "http://www.apem.com/int/index.php?controller=attachment&id_attachment=1371" (id 3) (at 145.288 30.226 0)
-      (effects (font (size 1.27 1.27)) hide)
-    )
-    (pin "1")
-    (pin "2")
-    (pin "3")
-    (pin "4")
-  )
   (symbol (lib_id "Device:LED_Small") (at 68.072 66.802 0) (mirror x) (unit 1)
     (in_bom yes) (on_board yes) (fields_autoplaced)
@@
     (property "Reference" "J101" (id 0) (at 106.045 148.844 0))
     (property "Value" "Conn_01x06_Male" (id 1) (at 106.045 151.384 0))
-    (property "Footprint" "" (id 2) (at 105.41 159.258 0)
+    (property "Footprint" "Connector_PinHeader_2.54mm:PinHeader_1x06_P2.54mm_Vertical" (id 2) (at 105.41 159.258 0)
       (effects (font (size 1.27 1.27)) hide)
     )
@@
     (pin "6")
   )
+  (symbol (lib_id "Connector:TestPoint") (at 209.804 69.342 0) (unit 1)
+    (in_bom yes) (on_board yes) (fields_autoplaced)
+    (property "Reference" "TP101" (id 0) (at 212.09 64.7699 0)
+      (effects (font (size 1.27 1.27)) (justify left))
+    )
+    (property "Value" "TestPoint" (id 1) (at 212.09 67.3099 0)
+      (effects (font (size 1.27 1.27)) (justify left))
+    )
+    (property "Footprint" "TestPoint:TestPoint_THTPad_D2.0mm_Drill1.0mm" (id 2) (at 214.884 69.342 0)
+      (effects (font (size 1.27 1.27)) hide)
+    )
+    (property "Datasheet" "~" (id 3) (at 214.884 69.342 0)
+      (effects (font (size 1.27 1.27)) hide)
+    )
+    (pin "1")
+  )
   (symbol (lib_id "Device:LED_Small") (at 48.26 53.34 180) (unit 1)
     (in_bom yes) (on_board yes) (fields_autoplaced)
@@
     (pin "1")
   )
-  (symbol (lib_id "Switch:SW_MEC_5E") (at 177.8 37.592 0) (unit 1)
-    (in_bom yes) (on_board yes) (fields_autoplaced)
-    (property "Reference" "SW102" (id 0) (at 177.8 27.178 0))
-    (property "Value" "SW_MEC_5E" (id 1) (at 177.8 29.718 0))
-    (property "Footprint" "Button_Switch_THT:SW_PUSH_6mm_H4.3mm" (id 2) (at 177.8 29.972 0)
-      (effects (font (size 1.27 1.27)) hide)
-    )
-    (property "Datasheet" "http://www.apem.com/int/index.php?controller=attachment&id_attachment=1371" (id 3) (at 177.8 29.972 0)
-      (effects (font (size 1.27 1.27)) hide)
-    )
-    (pin "1")
-    (pin "2")
-    (pin "3")
-    (pin "4")
-  )
   (symbol (lib_id "power:GND") (at 150.368 43.18 0) (unit 1)
     (in_bom yes) (on_board yes) (fields_autoplaced)
@@
     )
     (path "/bbb4eb0d-b2e0-418c-a1c7-628bb19d438f"
-      (reference "J101") (unit 1) (value "Conn_01x06_Male") (footprint "")
+      (reference "J101") (unit 1) (value "Conn_01x06_Male") (footprint "Connector_PinHeader_2.54mm:PinHeader_1x06_P2.54mm_Vertical")
     )
     (path "/03165e4a-9529-4bd2-b5e3-719f1aad0085"
-      (reference "J102") (unit 1) (value "Conn_01x10_Male") (footprint "")
+      (reference "J102") (unit 1) (value "Conn_01x10_Male") (footprint "Connector_PinHeader_2.54mm:PinHeader_1x10_P2.54mm_Vertical")
     )
     (path "/19a90198-4967-4abe-bb51-77933f224560"
-      (reference "J103") (unit 1) (value "Conn_01x04_Female") (footprint "")
-    )
-    (path "/9a18d167-9e04-400e-a0cd-f8dc367b9cbc"
-      (reference "SW101") (unit 1) (value "SW_MEC_5E") (footprint "Button_Switch_THT:SW_PUSH_6mm_H4.3mm")
-    )
-    (path "/ee5a251b-0002-4816-a8fd-dbb02a0adec4"
-      (reference "SW102") (unit 1) (value "SW_MEC_5E") (footprint "Button_Switch_THT:SW_PUSH_6mm_H4.3mm")
-    )
-  )
+      (reference "J103") (unit 1) (value "Conn_01x04_Female") (footprint "Connector_PinHeader_2.54mm:PinHeader_1x04_P2.54mm_Vertical")
+    )
+    (path "/348a9342-7ede-40fe-8e8e-c569bee6dccf"
+      (reference "SW101") (unit 1) (value "SW_SPST") (footprint "Button_Switch_THT:SW_PUSH_6mm_H4.3mm")
+    )
+    (path "/87aadc31-7606-4a81-8bbc-4ef15ccd9cbf"
+      (reference "SW102") (unit 1) (value "SW_SPST") (footprint "Button_Switch_THT:SW_PUSH_6mm_H4.3mm")
+    )
+    (path "/cbef01ce-e79f-4dde-9f7e-3742500e8d33"
+      (reference "TP101") (unit 1) (value "TestPoint") (footprint "TestPoint:TestPoint_THTPad_D2.0mm_Drill1.0mm")
+    )
+  )
